File: hardware/waterLevelController.kicad_sch (KiCad schematic)
At the start: 46 parts, among them J1 TerminalBlock, J2 Conn_01x02_Pin, J3 TerminalBlock, J4 Conn_01x03_Pin, J5 Conn_01x08_Pin, J6 Conn_01x05_Pin, J7 Conn_01x02_Pin, K1 SANYOU_SRD_Form_C, Q1 BC547, U1 ESP32-DevKit-V1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

Commit message: Gerber generated Version
Parts:
- J1: footprint TerminalBlock_MetzConnect:TerminalBlock_MetzConnect_Type011_RT05503HBLC_1x03_P5.00mm_Horizontal -> Connector_Phoenix_MC:PhoenixContact_MCV_1,5_3-G-3.81_1x03_P3.81mm_Vertical
- J3: footprint TerminalBlock:TerminalBlock_Altech_AK300-2_P5.00mm -> Connector_Phoenix_MC:PhoenixContact_MCV_1,5_2-G-3.81_1x02_P3.81mm_Vertical
- J6: footprint Connector_Samtec_HPM_THT:Samtec_HPM-05-01-x-S_Straight_1x05_Pitch5.08mm -> Connector_Phoenix_MC:PhoenixContact_MCV_1,5_5-G-3.81_1x05_P3.81mm_Vertical
Connections:
- net GND: now also J6.5 (Pin_5); no longer J6.1 (Pin_1)
- net ohtEmpty: now also J6.2 (Pin_2); no longer J6.4 (Pin_4)
- net ohtfull: now also J6.1 (Pin_1); no longer J6.5 (Pin_5)
- net ugtEmpty: now also J6.4 (Pin_4); no longer J6.2 (Pin_2)
- net at K1.1: now also J3.2 (Pin_2); no longer J3.1 (Pin_1)
- net at K1.3: now also J3.1 (Pin_1); no longer J3.2 (Pin_2)
Other:
- moved on the sheet: J3, J6
Changed lines of the file:
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@@
 	(wire
 		(pts
-			(xy 229.87 39.37) (xy 246.38 39.37)
+			(xy 246.38 24.13) (xy 246.38 30.48)
 		)
 		(stroke
@@
 	(wire
 		(pts
-			(xy 219.71 39.37) (xy 219.71 41.91)
+			(xy 229.87 39.37) (xy 246.38 39.37)
 		)
 		(stroke
@@
 	(wire
 		(pts
-			(xy 30.48 153.67) (xy 30.48 154.94)
+			(xy 219.71 39.37) (xy 219.71 41.91)
 		)
 		(stroke
@@
 	(wire
 		(pts
-			(xy 246.38 24.13) (xy 246.38 30.48)
+			(xy 30.48 153.67) (xy 30.48 154.94)
 		)
 		(stroke
@@
 	(wire
 		(pts
-			(xy 246.38 39.37) (xy 246.38 33.02)
-		)
-		(stroke
-			(width 0)
-			(type default)
-		)
-	)
-	(wire
-		(pts
 			(xy 132.08 118.11) (xy 144.78 118.11)
 		)
@@
 	(wire
 		(pts
+			(xy 246.38 33.02) (xy 246.38 39.37)
+		)
+		(stroke
+			(width 0)
+			(type default)
+		)
+	)
+	(wire
+		(pts
 			(xy 194.31 29.21) (xy 194.31 22.86)
 		)
@@
 			)
 		)
-		(property "Footprint" "TerminalBlock_MetzConnect:TerminalBlock_MetzConnect_Type011_RT05503HBLC_1x03_P5.00mm_Horizontal"
+		(property "Footprint" "Connector_Phoenix_MC:PhoenixContact_MCV_1,5_3-G-3.81_1x03_P3.81mm_Vertical"
 			(at 20.32 30.48 0)
 			(effects
@@
 	(symbol
 		(lib_id "Connector:Conn_01x05_Pin")
-		(at 80.01 170.18 180)
+		(at 80.01 170.18 0)
+		(mirror y)
 		(unit 1)
 		(exclude_from_sim no)
@@
 		(on_board yes)
 		(dnp no)
-		(fields_autoplaced yes)
 		(property "Reference" "J6"
-			(at 81.28 168.9099 0)
+			(at 81.28 171.4501 0)
 			(effects
 				(font
@@
 		)
 		(property "Value" "Conn_01x05_Pin"
-			(at 81.28 171.4499 0)
+			(at 81.28 168.9101 0)
 			(effects
 				(font
@@
 			)
 		)
-		(property "Footprint" "Connector_Samtec_HPM_THT:Samtec_HPM-05-01-x-S_Straight_1x05_Pitch5.08mm"
+		(property "Footprint" "Connector_Phoenix_MC:PhoenixContact_MCV_1,5_5-G-3.81_1x05_P3.81mm_Vertical"
 			(at 80.01 170.18 0)
 			(effects
@@
 	(symbol
 		(lib_id "Connector:Conn_01x02_Pin")
-		(at 251.46 33.02 180)
+		(at 251.46 30.48 0)
+		(mirror y)
 		(unit 1)
 		(exclude_from_sim no)
@@
 		(dnp no)
 		(property "Reference" "J3"
-			(at 253.492 38.1 0)
+			(at 253.492 25.4 0)
 			(effects
 				(font
@@
 		)
 		(property "Value" "TerminalBlock"
-			(at 254.762 35.814 0)
+			(at 254.762 27.686 0)
 			(effects
 				(font
@@
 			)
 		)
-		(property "Footprint" "TerminalBlock:TerminalBlock_Altech_AK300-2_P5.00mm"
-			(at 251.46 33.02 0)
+		(property "Footprint" "Connector_Phoenix_MC:PhoenixContact_MCV_1,5_2-G-3.81_1x02_P3.81mm_Vertical"
+			(at 251.46 30.48 0)
 			(effects
 				(font
@@
 		)
 		(property "Datasheet" "~"
-			(at 251.46 33.02 0)
+			(at 251.46 30.48 0)
 			(effects
 				(font
@@
 		)
 		(property "Description" "Generic connector, single row, 01x02, script generated"
-			(at 251.46 33.02 0)
+			(at 251.46 30.48 0)
 			(effects
 				(font
