File: hardware/waterLevelController.kicad_pcb (KiCad board)
At the start: 2 copper layers, 84 x 95 mm, 46 parts, among them J1 TerminalBlock, J2 Conn_01x02_Pin, J3 TerminalBlock, J4 Conn_01x03_Pin, J5 Conn_01x08_Pin, J6 Conn_01x05_Pin, J7 Conn_01x02_Pin, K1 SANYOU_SRD_Form_C, Q1 BC547, U1 ESP32-DevKit-V1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

Commit message: Gerber generated Version
Parts:
- J1: footprint TerminalBlock_MetzConnect:TerminalBlock_MetzConnect_Type011_RT05503HBLC_1x03_P5.00mm_Horizontal -> Connector_Phoenix_MC:PhoenixContact_MCV_1,5_3-G-3.81_1x03_P3.81mm_Vertical
- J3: footprint TerminalBlock:TerminalBlock_Altech_AK300-2_P5.00mm -> Connector_Phoenix_MC:PhoenixContact_MCV_1,5_2-G-3.81_1x02_P3.81mm_Vertical
- J6: footprint Connector_Samtec_HPM_THT:Samtec_HPM-05-01-x-S_Straight_1x05_Pitch5.08mm -> Connector_Phoenix_MC:PhoenixContact_MCV_1,5_5-G-3.81_1x05_P3.81mm_Vertical
- moved J6 18.3 mm to (48.0, 60.9), turned to -90 degrees
- moved J3 5.02 mm to (116.4, 20.9), turned to 180 degrees
- moved J1 2.44 mm to (47.5, 24.7)
- moved J2 1.84 mm to (51.0, 107.0)
- moved C2 1.75 mm to (46.0, 102.0)
- moved C7 1.75 mm to (51.5, 102.0)
- moved R3 1.75 mm to (46.8, 92.9)
- moved R5 1.75 mm to (50.8, 97.1)
Connections:
- J6 pad 1: GND -> ohtfull
- J6 pad 2: ugtEmpty -> ohtEmpty
- J6 pad 4: ohtEmpty -> ugtEmpty
- J6 pad 5: ohtfull -> GND
- K1 pad 1: Net-(J3-Pin_1) -> Net-(J3-Pin_2)
- K1 pad 3: Net-(J3-Pin_2) -> Net-(J3-Pin_1)
Routing:
- net Net-(J2-Pin_2): track 23.6 -> 27.7 mm
- net Net-(J3-Pin_1): track 20.7 -> 24.3 mm
- net +3.3V: track 107.8 -> 104.5 mm
- net ohtfull: track 28.1 -> 30.7 mm
- net Net-(D2-A): track 10.0 -> 7.93 mm
- net Net-(D1-A): track 10.0 -> 8.42 mm
- net i_sens: track 52.9 -> 51.4 mm
- net ohtEmpty: track 33.6 -> 34.9 mm
Other:
- board size 84 x 95 mm -> 81 x 95 mm

Commit message: silkscreen updated
Other:
- board text added: "oht-full oht-empty ugt-full ugt-empty Gnd"
- board text removed: "oht-full oht-empty ugt-full ugt-empty"
Changed lines of the file:
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@@
 		(tags "C Disc series Radial pin pitch 2.50mm diameter 3.8mm width 2.6mm Capacitor")
 		(property "Reference" "C4"
-			(at 1.94 2.9325 180)
+			(at 5.25 0 180)
 			(layer "F.SilkS")
 			(effects
@@
 		(tags "Resistor Axial_DIN0309 series Axial Vertical pin pitch 5.08mm 0.5W = 1/2W length 9mm diameter 3.2mm")
 		(property "Reference" "R15"
-			(at 7.5725 -2.44 0)
+			(at 8.0725 0.06 0)
 			(layer "F.SilkS")
 			(effects
@@
 		(tags "Resistor Axial_DIN0309 series Axial Vertical pin pitch 5.08mm 0.5W = 1/2W length 9mm diameter 3.2mm")
 		(property "Reference" "R13"
-			(at 7.8225 -1.85 0)
+			(at 7.8225 0.06 0)
 			(layer "F.SilkS")
 			(effects
@@
 		(tags "Resistor Axial_DIN0309 series Axial Vertical pin pitch 5.08mm 0.5W = 1/2W length 9mm diameter 3.2mm")
 		(property "Reference" "R18"
-			(at 8.2075 1.94 0)
+			(at 8.2075 -0.06 0)
 			(layer "F.SilkS")
 			(effects
@@
 		(tags "C Disc series Radial pin pitch 2.50mm diameter 3.8mm width 2.6mm Capacitor")
 		(property "Reference" "C7"
-			(at 5.25 0 0)
+			(at 4.5 0 0)
 			(layer "F.SilkS")
 			(effects
@@
 		(tags "Through hole pin header THT 1x02 2.54mm single row")
 		(property "Reference" "J7"
-			(at 0 -2.38 90)
+			(at 0 -3.225 180)
 			(layer "F.SilkS")
 			(effects
@@
 		(tags "Resistor Axial_DIN0309 series Axial Vertical pin pitch 5.08mm 0.5W = 1/2W length 9mm diameter 3.2mm")
 		(property "Reference" "R2"
-			(at 5.64 -4.5 180)
+			(at 7.14 0 180)
 			(layer "F.SilkS")
 			(effects
@@
 		(tags "Resistor Axial_DIN0309 series Axial Vertical pin pitch 5.08mm 0.5W = 1/2W length 9mm diameter 3.2mm")
 		(property "Reference" "R5"
-			(at 7.14 -5.5 180)
+			(at 7.14 -0.25 180)
 			(layer "F.SilkS")
 			(effects
@@
 		(tags "Resistor Axial_DIN0309 series Axial Vertical pin pitch 5.08mm 0.5W = 1/2W length 9mm diameter 3.2mm")
 		(property "Reference" "R4"
-			(at 2.54 -2.72 0)
+			(at 7.36 0 0)
 			(layer "F.SilkS")
 			(effects
@@
 		(tags "C Radial series Radial pin pitch 5.00mm diameter 12.5mm height 20mm Non-Polar Electrolytic Capacitor")
 		(property "Reference" "C1"
-			(at 1.5 -12 180)
+			(at -6 0 180)
 			(layer "F.SilkS")
 			(effects
@@
 		(tags "Resistor Axial_DIN0309 series Axial Vertical pin pitch 5.08mm 0.5W = 1/2W length 9mm diameter 3.2mm")
 		(property "Reference" "R8"
-			(at 2.54 -2.72 0)
+			(at -2.9275 0 0)
 			(layer "F.SilkS")
 			(effects
@@
 		(tags "CP Radial series Radial pin pitch 2.50mm diameter 8mm height 10mm Electrolytic Capacitor")
 		(property "Reference" "C3"
-			(at 1.25 -5.25 180)
+			(at -0.5 -5.5 180)
 			(layer "F.SilkS")
 			(effects
@@
 		(tags "Resistor Axial_DIN0309 series Axial Vertical pin pitch 5.08mm 0.5W = 1/2W length 9mm diameter 3.2mm")
 		(property "Reference" "R1"
-			(at 6.13 3 180)
+			(at 7.08 0 180)
 			(layer "F.SilkS")
 			(effects
@@
 		(tags "to-92 sc-43 sc-43a sot54 PA33 transistor")
 		(property "Reference" "Q1"
-			(at 0.27 -5.36 0)
+			(at -2.23 -3.36 0)
 			(layer "F.SilkS")
 			(effects
@@
 		(tags "Resistor Axial_DIN0309 series Axial Vertical pin pitch 5.08mm 0.5W = 1/2W length 9mm diameter 3.2mm")
 		(property "Reference" "R17"
-			(at 8.1475 1.44 0)
+			(at 8.1475 -0.06 0)
 			(layer "F.SilkS")
 			(effects
@@
 		(tags "Resistor Axial_DIN0309 series Axial Vertical pin pitch 5.08mm 0.5W = 1/2W length 9mm diameter 3.2mm")
 		(property "Reference" "R10"
-			(at -3.4275 -1.94 0)
+			(at 7.5725 0 0)
 			(layer "F.SilkS")
 			(effects
@@
 		(tags "LED")
 		(property "Reference" "D3"
-			(at 0.77 5.5 180)
+			(at 1.27 -4 180)
 			(layer "F.SilkS")
 			(effects
@@
 		(tags "Resistor Axial_DIN0309 series Axial Vertical pin pitch 5.08mm 0.5W = 1/2W length 9mm diameter 3.2mm")
 		(property "Reference" "R3"
-			(at -0.86 -7 180)
+			(at -2.86 -0.25 180)
 			(layer "F.SilkS")
 			(effects
@@
 		(tags "Diode DO-41_SOD81 series Axial Horizontal pin pitch 10.16mm  length 5.2mm diameter 2.7mm")
 		(property "Reference" "D1"
-			(at -2.92 -2.5 0)
+			(at -2.92 0 0)
 			(layer "F.SilkS")
 			(effects
@@
 		(tags "Resistor Axial_DIN0309 series Axial Vertical pin pitch 5.08mm 0.5W = 1/2W length 9mm diameter 3.2mm")
 		(property "Reference" "R14"
-			(at 7.8225 -2.15 0)
+			(at 7.8225 0.06 0)
 			(layer "F.SilkS")
 			(effects
@@
 		(tags "Resistor Axial_DIN0309 series Axial Vertical pin pitch 5.08mm 0.5W = 1/2W length 9mm diameter 3.2mm")
 		(property "Reference" "R12"
-			(at 7.5725 -0.69 0)
+			(at 7.5725 0.06 0)
 			(layer "F.SilkS")
 			(effects
@@
 		(tags "Resistor Axial_DIN0309 series Axial Vertical pin pitch 5.08mm 0.5W = 1/2W length 9mm diameter 3.2mm")
 		(property "Reference" "R19"
-			(at 8.2075 1.94 0)
+			(at 8.2075 -0.06 0)
 			(layer "F.SilkS")
 			(effects
@@
 		(tags "Resistor Axial_DIN0309 series Axial Vertical pin pitch 5.08mm 0.5W = 1/2W length 9mm diameter 3.2mm")
 		(property "Reference" "R9"
-			(at -3.6775 -1.85 0)
+			(at 7.5725 0 0)
 			(layer "F.SilkS")
 			(effects
@@
 		(tags "Resistor Axial_DIN0309 series Axial Vertical pin pitch 5.08mm 0.5W = 1/2W length 9mm diameter 3.2mm")
 		(property "Reference" "R16"
-			(at 8.2075 0.44 0)
+			(at 8.2075 -0.06 0)
 			(layer "F.SilkS")
 			(effects
@@
 		(tags "Resistor Axial_DIN0309 series Axial Vertical pin pitch 5.08mm 0.5W = 1/2W length 9mm diameter 3.2mm")
 		(property "Reference" "R7"
-			(at 2.54 -2.72 0)
+			(at -3.4275 0 0)
 			(layer "F.SilkS")
 			(effects
@@
 		(tags "Resistor Axial_DIN0309 series Axial Vertical pin pitch 5.08mm 0.5W = 1/2W length 9mm diameter 3.2mm")
 		(property "Reference" "R6"
-			(at -3 3 180)
+			(at -3 0 180)
 			(layer "F.SilkS")
 			(effects
@@
 		(tags "C Disc series Radial pin pitch 2.50mm diameter 3.8mm width 2.6mm Capacitor")
 		(property "Reference" "C5"
-			(at 5 -2 180)
+			(at 5 0 180)
 			(layer "F.SilkS")
 			(effects
@@
 		(tags "Resistor Axial_DIN0309 series Axial Vertical pin pitch 5.08mm 0.5W = 1/2W length 9mm diameter 3.2mm")
 		(property "Reference" "R11"
-			(at -3.6775 -1.85 0)
+			(at 7.5725 0 0)
 			(layer "F.SilkS")
 			(effects
@@
 		(tags "C Disc series Radial pin pitch 2.50mm diameter 3.8mm width 2.6mm Capacitor")
 		(property "Reference" "C2"
-			(at 0.5 -2.5 0)
+			(at -2 0 0)
 			(layer "F.SilkS")
 			(effects
@@
 	)
 	(gr_text "Alarm\nPower\npump On/Off"
-		(at 112 54 0)
+		(at 113.5 65 0)
 		(layer "F.SilkS")
 		(effects
@@
 	)
 	(gr_text "CT"
-		(at 44.25 106.5 0)
+		(at 44.5 107 0)
 		(layer "F.SilkS")
 		(effects
@@
 		)
 	)
-	(gr_text "oht-full\noht-empty\nugt-full\nugt-empty"
-		(at 45.5 50.5 0)
+	(gr_text "oht-full\noht-empty\nugt-full\nugt-empty\nGnd"
+		(at 45 55.5 0)
 		(layer "F.SilkS")
 		(effects
@@
 	)
 	(segment
-		(start 106.7 81.3275)
-		(end 106.7 99.5)
+		(start 104.8725 79.5)
+		(end 106.7 81.3275)
 		(width 0.75)
 		(layer "B.Cu")
@@
 	)
 	(segment
-		(start 104.8725 79.5)
-		(end 106.7 81.3275)
+		(start 92.9325 77.32)
+		(end 99.494025 77.32)
 		(width 0.75)
 		(layer "B.Cu")
@@
 	)
 	(segment
-		(start 99.439 79.5)
-		(end 104.8725 79.5)
+		(start 99.494025 77.32)
+		(end 101.674025 79.5)
 		(width 0.75)
 		(layer "B.Cu")
@@
 	)
 	(segment
-		(start 97.259 77.32)
-		(end 99.439 79.5)
+		(start 106.7 81.3275)
+		(end 106.7 99.5)
 		(width 0.75)
 		(layer "B.Cu")
@@
 	)
 	(segment
-		(start 92.9325 77.32)
-		(end 97.259 77.32)
+		(start 101.674025 79.5)
+		(end 104.8725 79.5)
 		(width 0.75)
 		(layer "B.Cu")
